File: hardware/accelerometer-v2.kicad_pcb (KiCad board)
At the start: 2 copper layers, 20 x 25 mm, 25 parts, among them P1 CON-SENSOR, P2 Debug, P3 Boot, U1 XMC1302, U2 KX122-1037, U3 DRILL, U4 DRILL, U5 DRILL, U6 DRILL

Commit message: specify processor as xmc1100
Parts:
- U1: value XMC1302 -> XMC1100
Changed lines of the file:
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@@
       (effects (font (size 0.3 0.3) (thickness 0.075)))
     )
-    (fp_text value XMC1302 (at 0 0.8 180) (layer F.Fab)
+    (fp_text value XMC1100 (at 0 0.8 180) (layer F.Fab)
       (effects (font (size 0.3 0.3) (thickness 0.075)))
     )

Commit message: fix library settings
Other:
- net class Default removed
